File: WingManPCB.sch (KiCad schematic (older format))
At the start: 1 part

Commit message: Beginning the schematic work
Parts:
- removed U?: ATmega32A-AU, Package_QFP:TQFP-44_10x10mm_P0.8mm, symbol MCU_Microchip_ATmega:ATmega32A-AU
- added C?: 1u, symbol Device:C_Small
- added C? (x2): 22p, symbol Device:C_Small
- added C? (x4): 0.1u, symbol Device:C_Small
- added C?: 10u, symbol Device:C_Small
- added MX? (x6): MX-NoLED, symbol MX_Alps_Hybrid:MX-NoLED
- added R? (x2): 10k, symbol Device:R_Small
- added S?: SW_SKQG, symbol localfootprints:SW_SKQG
- added U?: ATmega32U4-AU, Package_QFP:TQFP-44_10x10mm_P0.8mm, symbol MCU_Microchip_ATmega:ATmega32U4-AU
- added Y?: Crystal_GND24_Small, symbol Device:Crystal_GND24_Small
Connections:
- new net: R?.2, U?.33 (~HWB~/PE2)
- new net: C?.1, U?.6 (UCAP)
- new net +5V: C?.1, C?.1, C?.1, C?.1, C?.1, R?.1, U?.14 (VCC), U?.2 (UVCC), U?.24 (AVCC), U?.34 (VCC), U?.44 (AVCC)
- new net DM: U?.3 (D-)
- new net DP: U?.4 (D+)
- new net GND: C?.2, C?.2, C?.2, C?.2, C?.2, C?.2, C?.2, C?.2, R?.1, S?.2, U?.15 (GND), U?.23 (GND), U?.35 (GND), U?.43 (GND), U?.5 (UGND), Y?.2, Y?.4
- new net RESET: R?.2, S?.1, U?.13 (~RESET)
- new net XTAL1: C?.1, U?.17 (XTAL1), Y?.1
- new net XTAL2: C?.1, U?.16 (XTAL2), Y?.3
- no-connect marks 0 -> 4

Commit message: Schematic complete
Parts:
- added D1: PRTR5V0U2X, Package_TO_SOT_SMD:SOT-143, symbol Power_Protection:PRTR5V0U2X
- added D2, D3, D4, D5, D6, D7: D_Small, Diode_SMD:D_SOD-123, symbol Device:D_Small
- added F1: 500m, Fuse:Fuse_1206_3216Metric, symbol Device:Polyfuse_Small
- added R1, R2: 22, Resistor_SMD:R_0805_2012Metric, symbol Device:R_Small
- added R3, R4: 5.1k, Resistor_SMD:R_0805_2012Metric, symbol Device:R_Small
- added USB1: HRO-TYPE-C-31-M-12, Type-C:HRO-TYPE-C-31-M-12-Assembly, symbol Type-C:HRO-TYPE-C-31-M-12
- C1, C2, C3, C4, C5, C6, C7, C8: renamed from C?; footprint (none) -> Capacitor_SMD:C_0805_2012Metric
- MX1, MX2, MX3, MX4, MX5: renamed from MX?; footprint (none) -> MX_Only:MXOnly-1U
- MX6: renamed from MX?; footprint (none) -> Resistor_SMD:R_0805_2012Metric
- R5, R6: renamed from R?; footprint (none) -> Resistor_SMD:R_0805_2012Metric
- S1: renamed from S?; footprint (none) -> random-keyboard-parts:SKQG-1155865
- Y1: renamed from Y?; footprint (none) -> Crystal:Crystal_SMD_3225-4Pin_3.2x2.5mm
- gave numbers to parts that had none: 1
Connections:
- net +5V: now also F1.1
- net DP: now also R2.2
- net GND: now also D1.1 (GND), R3.1, R4.1, USB1.1 (GND), USB1.12 (GND), USB1.13 (SHIELD)
- net COL0: now reaches MX1.1 (COL)
- net at MX1.2 (ROW): now also D2.2 (A)
- net COL1: now reaches MX2.1 (COL)
- net at MX2.2 (ROW): now also D3.2 (A)
- net COL2: now reaches MX3.1 (COL)
- net at MX3.2 (ROW): now also D4.2 (A)
- net COL3: now reaches MX4.1 (COL)
- net at MX4.2 (ROW): now also D5.2 (A)
- net COL4: now reaches MX5.1 (COL)
- net at MX5.2 (ROW): now also D6.2 (A)
- net COL5: now reaches MX6.1 (COL)
- net at MX6.2 (ROW): now also D7.2 (A)
- new net: R3.2, USB1.10 (CC2)
- new net: R4.2, USB1.4 (CC1)
- new net: D1.3 (I/O2), R1.1, USB1.5 (DN2), USB1.7 (DN1)
- new net: D1.2 (I/O1), R2.1, USB1.6 (DP1), USB1.8 (DP2)
- new net DN: R1.2
- new net ROW0: D2.1 (K), D3.1 (K), D4.1 (K), D5.1 (K), D6.1 (K), D7.1 (K)
- new net VCC: D1.4 (VCC), F1.2, USB1.11 (VBUS), USB1.2 (VBUS)
- no-connect marks 4 -> 6
Other:
- moved on the sheet: MX1, MX2, MX3, MX5, MX6

Commit message: Sch complete, matrix routed, components mostly placed
Parts:
- removed S1: SW_SKQG, random-keyboard-parts:SKQG-1155865, symbol localfootprints:SW_SKQG
- added SW1: SW_Push, Button_Switch_SMD:SW_SPST_SKQG_WithStem, symbol Switch:SW_Push
- MX1, MX2, MX3, MX4, MX5: footprint MX_Only:MXOnly-1U -> MX_Only:MXOnly-1U-NoLED
- MX6: footprint Resistor_SMD:R_0805_2012Metric -> MX_Only:MXOnly-1U-NoLED
Connections:
- net DM is gone; now on net DN: U1.3 (D-)
- net +5V: now also U1.7 (VBUS)
- net COL0: now also U1.31 (PC6)
- net COL1: now also U1.30 (PB6)
- net COL2: now also U1.29 (PB5)
- net COL3: now also U1.28 (PB4)
- net COL4: now also U1.27 (PD7)
- net COL5: now also U1.26 (PD6)
- net GND: now also SW1.1
- net ROW0: now also U1.32 (PC7)
- net RESET: no longer names the net of R6.2, U1.13 (~RESET)
- net RESET: now also SW1.2
- no-connect marks 6 -> 3
Other:
- moved on the sheet: R6
Changed lines of the file:
@@
 F 0 "MX1" H 2233 6073 60  0000 C CNN
 F 1 "MX-NoLED" H 2233 5999 20  0000 C CNN
-F 2 "MX_Only:MXOnly-1U" H 1575 5825 60  0001 C CNN
+F 2 "MX_Only:MXOnly-1U-NoLED" H 1575 5825 60  0001 C CNN
 F 3 "" H 1575 5825 60  0001 C CNN
 	1    2200 5850
@@
 F 0 "MX2" H 2683 6073 60  0000 C CNN
 F 1 "MX-NoLED" H 2683 5999 20  0000 C CNN
-F 2 "MX_Only:MXOnly-1U" H 2025 5825 60  0001 C CNN
+F 2 "MX_Only:MXOnly-1U-NoLED" H 2025 5825 60  0001 C CNN
 F 3 "" H 2025 5825 60  0001 C CNN
 	1    2650 5850
@@
 F 0 "MX3" H 3133 6073 60  0000 C CNN
 F 1 "MX-NoLED" H 3133 5999 20  0000 C CNN
-F 2 "MX_Only:MXOnly-1U" H 2475 5825 60  0001 C CNN
+F 2 "MX_Only:MXOnly-1U-NoLED" H 2475 5825 60  0001 C CNN
 F 3 "" H 2475 5825 60  0001 C CNN
 	1    3100 5850
@@
 F 0 "MX4" H 3583 6073 60  0000 C CNN
 F 1 "MX-NoLED" H 3583 5999 20  0000 C CNN
-F 2 "MX_Only:MXOnly-1U" H 2925 5825 60  0001 C CNN
+F 2 "MX_Only:MXOnly-1U-NoLED" H 2925 5825 60  0001 C CNN
 F 3 "" H 2925 5825 60  0001 C CNN
 	1    3550 5850
@@
 F 0 "MX5" H 4033 6073 60  0000 C CNN
 F 1 "MX-NoLED" H 4033 5999 20  0000 C CNN
-F 2 "MX_Only:MXOnly-1U" H 3375 5825 60  0001 C CNN
+F 2 "MX_Only:MXOnly-1U-NoLED" H 3375 5825 60  0001 C CNN
 F 3 "" H 3375 5825 60  0001 C CNN
 	1    4000 5850
@@
 F 0 "MX6" H 4483 6073 60  0000 C CNN
 F 1 "MX-NoLED" H 4483 5999 20  0000 C CNN
-F 2 "Resistor_SMD:R_0805_2012Metric" H 3825 5825 60  0001 C CNN
+F 2 "MX_Only:MXOnly-1U-NoLED" H 3825 5825 60  0001 C CNN
 F 3 "" H 3825 5825 60  0001 C CNN
 	1    4450 5850
@@
 Text GLabel 8700 2000 0    50   Input ~ 0
 XTAL2
-Text GLabel 8700 1600 0    50   Input ~ 0
-RESET
 Text GLabel 8700 2600 0    50   Input ~ 0
 DP
 Text GLabel 8700 2700 0    50   Input ~ 0
-DM
+DN
 $Comp
 L Device:R_Small R5
@@
 	6200 3350 6500 3350
 $Comp
-L localfootprints:SW_SKQG S1
-U 1 1 60800A03
-P 5900 4300
-F 0 "S1" H 5900 4525 50  0000 C CNN
-F 1 "SW_SKQG" H 5900 4434 50  0000 C CNN
-F 2 "random-keyboard-parts:SKQG-1155865" H 5900 4450 50  0001 C CNN
-F 3 "" H 5900 4450 50  0001 C CNN
-	1    5900 4300
-	1    0    0    -1
-$EndComp
-NoConn ~ 6300 4800
-$Comp
 L Device:R_Small R6
 U 1 1 60803720
-P 6500 4050
-F 0 "R6" H 6559 4096 50  0000 L CNN
-F 1 "10k" H 6559 4005 50  0000 L CNN
-F 2 "Resistor_SMD:R_0805_2012Metric" H 6500 4050 50  0001 C CNN
-F 3 "~" H 6500 4050 50  0001 C CNN
-	1    6500 4050
+P 8450 1300
+F 0 "R6" H 8509 1346 50  0000 L CNN
+F 1 "10k" H 8509 1255 50  0000 L CNN
+F 2 "Resistor_SMD:R_0805_2012Metric" H 8450 1300 50  0001 C CNN
+F 3 "~" H 8450 1300 50  0001 C CNN
+	1    8450 1300
 	1    0    0    -1
 $EndComp
@@
 L power:+5V #PWR05
 U 1 1 608045C8
-P 6500 3950
-F 0 "#PWR05" H 6500 3800 50  0001 C CNN
-F 1 "+5V" H 6515 4123 50  0000 C CNN
-F 2 "" H 6500 3950 50  0001 C CNN
-F 3 "" H 6500 3950 50  0001 C CNN
-	1    6500 3950
-	1    0    0    -1
-$EndComp
-Wire Wire Line
-	6500 4150 6500 4300
-Wire Wire Line
-	6500 4300 6300 4300
-Wire Wire Line
-	6500 4300 6750 4300
-Connection ~ 6500 4300
-Text GLabel 6750 4300 2    50   Input ~ 0
-RESET
-NoConn ~ 5700 4300
-NoConn ~ 5500 4300
+P 8450 1200
+F 0 "#PWR05" H 8450 1050 50  0001 C CNN
+F 1 "+5V" H 8465 1373 50  0000 C CNN
+F 2 "" H 8450 1200 50  0001 C CNN
+F 3 "" H 8450 1200 50  0001 C CNN
+	1    8450 1200
+	1    0    0    -1
+$EndComp
 $Comp
 L power:GND #PWR06
 U 1 1 6080A20A
-P 5400 4900
-F 0 "#PWR06" H 5400 4650 50  0001 C CNN
-F 1 "GND" H 5405 4727 50  0000 C CNN
-F 2 "" H 5400 4900 50  0001 C CNN
-F 3 "" H 5400 4900 50  0001 C CNN
-	1    5400 4900
-	1    0    0    -1
-$EndComp
-Wire Wire Line
-	5500 4800 5400 4800
-Wire Wire Line
-	5400 4800 5400 4900
+P 7900 1700
+F 0 "#PWR06" H 7900 1450 50  0001 C CNN
+F 1 "GND" H 7905 1527 50  0000 C CNN
+F 2 "" H 7900 1700 50  0001 C CNN
+F 3 "" H 7900 1700 50  0001 C CNN
+	1    7900 1700
+	1    0    0    -1
+$EndComp
 $Comp
 L Type-C:HRO-TYPE-C-31-M-12 USB1
@@
 Connection ~ 2000 1350
 Wire Wire Line
-	2000 1350 2200 1350
+	2000 1350 2100 1350
 Wire Wire Line
 	1800 1650 2200 1650
@@
 	0    -1   -1   0
 $EndComp
-Wire Wire Line
-	3950 1850 4100 1850
 $Comp
 L Device:R_Small R2
@@
 $EndComp
 Wire Wire Line
-	3300 1350 3000 1350
+	3300 1350 3150 1350
 NoConn ~ 1800 1450
 NoConn ~ 1800 2050
@@
 Connection ~ 1900 2450
 Wire Wire Line
-	2350 2450 2000 2450
+	2350 2450 2150 2450
 Connection ~ 2000 2450
 Wire Wire Line
@@
 Wire Wire Line
 	3750 2600 3750 3050
-Connection ~ 3450 1850
-Wire Wire Line
-	3450 1850 3750 1850
 Wire Wire Line
 	2900 1950 2900 2600
@@
 Text GLabel 4600 5500 1    50   Input ~ 0
 COL5
+Wire Wire Line
+	4100 1850 3950 1850
+Wire Wire Line
+	3750 1850 3450 1850
+Connection ~ 3450 1850
+$Comp
+L power:PWR_FLAG #FLG0101
+U 1 1 608AEF18
+P 3150 1350
+F 0 "#FLG0101" H 3150 1425 50  0001 C CNN
+F 1 "PWR_FLAG" H 3150 1523 50  0000 C CNN
+F 2 "" H 3150 1350 50  0001 C CNN
+F 3 "~" H 3150 1350 50  0001 C CNN
+	1    3150 1350
+	1    0    0    -1
+$EndComp
+Connection ~ 3150 1350
+Wire Wire Line
+	3150 1350 3000 1350
+$Comp
+L power:PWR_FLAG #FLG0102
+U 1 1 608B0697
+P 2100 1350
+F 0 "#FLG0102" H 2100 1425 50  0001 C CNN
+F 1 "PWR_FLAG" H 2100 1523 50  0000 C CNN
+F 2 "" H 2100 1350 50  0001 C CNN
+F 3 "~" H 2100 1350 50  0001 C CNN
+	1    2100 1350
+	1    0    0    -1
+$EndComp
+Connection ~ 2100 1350
+Wire Wire Line
+	2100 1350 2200 1350
+$Comp
+L power:PWR_FLAG #FLG0103
+U 1 1 608B1985
+P 2150 2450
+F 0 "#FLG0103" H 2150 2525 50  0001 C CNN
+F 1 "PWR_FLAG" H 2150 2623 50  0000 C CNN
+F 2 "" H 2150 2450 50  0001 C CNN
+F 3 "~" H 2150 2450 50  0001 C CNN
+	1    2150 2450
+	-1   0    0    1
+$EndComp
+Connection ~ 2150 2450
+Wire Wire Line
+	2150 2450 2000 2450
+Text GLabel 9900 2600 2    50   Input ~ 0
+ROW0
+Text GLabel 9900 2500 2    50   Input ~ 0
+COL0
+Text GLabel 9900 2200 2    50   Input ~ 0
+COL1
+Text GLabel 9900 2100 2    50   Input ~ 0
+COL2
+Text GLabel 9900 2000 2    50   Input ~ 0
+COL3
+Text GLabel 9900 3500 2    50   Input ~ 0
+COL4
+Text GLabel 9900 3400 2    50   Input ~ 0
+COL5
+Wire Wire Line
+	8700 2400 8200 2400
+Wire Wire Line
+	8200 2400 8200 2300
+$Comp
+L power:+5V #PWR0108
+U 1 1 608C9C0D
+P 8200 2300
+F 0 "#PWR0108" H 8200 2150 50  0001 C CNN
+F 1 "+5V" H 8215 2473 50  0000 C CNN
+F 2 "" H 8200 2300 50  0001 C CNN
+F 3 "" H 8200 2300 50  0001 C CNN
+	1    8200 2300
+	1    0    0    -1
+$EndComp
+$Comp
+L Switch:SW_Push SW1
+U 1 1 608CB4D3
+P 8150 1600
+F 0 "SW1" H 8150 1885 50  0000 C CNN
+F 1 "SW_Push" H 8150 1794 50  0000 C CNN
+F 2 "Button_Switch_SMD:SW_SPST_SKQG_WithStem" H 8150 1800 50  0001 C CNN
+F 3 "~" H 8150 1800 50  0001 C CNN
+	1    8150 1600
+	1    0    0    -1
+$EndComp
+Wire Wire Line
+	8700 1600 8450 1600
+Wire Wire Line
+	8450 1400 8450 1600
+Connection ~ 8450 1600
+Wire Wire Line
+	8450 1600 8350 1600
+Wire Wire Line
+	7950 1600 7900 1600
+Wire Wire Line
+	7900 1600 7900 1700
 $EndSCHEMATC
